File: kicad/motordrivershield.sch (KiCad schematic (older format))
At the start: 37 parts, among them CN1 ARDUINO_MKR, CN2 QWIIC, P1 CONN_01X03, P2 CONN_01X03, U1 PCA9685_TSSOP28, U2 ADS1015

Commit message: added 5V to arduino header
Parts:
- added L? (x3): Label, symbol devices:Label
Connections:
- net +5V: now also CN1.28 (5V0)
- no-connect marks 29 -> 28
Other:
- moved on the sheet: CN1, JP10, JP9
Changed lines of the file:
@@
 L MODULE_compute:ARDUINO_MKR CN1
 U 1 1 5F5E81F1
-P 3650 1750
-F 0 "CN1" H 3650 2647 60  0000 C CNN
-F 1 "ARDUINO_MKR" H 3650 2541 60  0000 C CNN
-F 2 "MODULE_compute:ARDUINO_MKR" H 3550 2400 60  0001 C CNN
-F 3 "" H 3650 1450 60  0000 C CNN
-	1    3650 1750
+P 2350 1850
+F 0 "CN1" H 2350 2747 60  0000 C CNN
+F 1 "ARDUINO_MKR" H 2350 2641 60  0000 C CNN
+F 2 "MODULE_compute:ARDUINO_MKR" H 2250 2500 60  0001 C CNN
+F 3 "" H 2350 1550 60  0000 C CNN
+	1    2350 1850
 	1    0    0    -1
 $EndComp
@@
 $EndComp
 Wire Wire Line
-	4250 1400 4500 1400
-Wire Wire Line
-	4500 1400 4500 1500
-Wire Wire Line
-	4250 1300 4500 1300
-Wire Wire Line
-	4500 1300 4500 1200
+	2950 1500 3200 1500
+Wire Wire Line
+	3200 1500 3200 1600
+Wire Wire Line
+	2950 1400 3200 1400
+Wire Wire Line
+	3200 1400 3200 1300
 $Comp
 L power-supply:+3V3 #PWR0112
 U 1 1 5F67ACD5
-P 4500 1200
-F 0 "#PWR0112" H 4500 1050 50  0001 C CNN
-F 1 "+3V3" H 4515 1373 50  0000 C CNN
-F 2 "" H 4500 1200 50  0000 C CNN
-F 3 "" H 4500 1200 50  0000 C CNN
-	1    4500 1200
+P 3200 1300
+F 0 "#PWR0112" H 3200 1150 50  0001 C CNN
+F 1 "+3V3" H 3215 1473 50  0000 C CNN
+F 2 "" H 3200 1300 50  0000 C CNN
+F 3 "" H 3200 1300 50  0000 C CNN
+	1    3200 1300
 	1    0    0    -1
 $EndComp
@@
 L power-supply:GND #PWR0113
 U 1 1 5F67DE8B
-P 4500 1500
-F 0 "#PWR0113" H 4500 1250 50  0001 C CNN
-F 1 "GND" H 4505 1327 50  0000 C CNN
-F 2 "" H 4500 1500 50  0000 C CNN
-F 3 "" H 4500 1500 50  0000 C CNN
-	1    4500 1500
-	1    0    0    -1
-$EndComp
-Wire Wire Line
-	3050 2300 2650 2300
-Wire Wire Line
-	3050 2400 2650 2400
-Wire Wire Line
-	4250 1900 4650 1900
-Wire Wire Line
-	4250 1800 4650 1800
-Text Label 2650 2300 0    50   ~ 0
+P 3200 1600
+F 0 "#PWR0113" H 3200 1350 50  0001 C CNN
+F 1 "GND" H 3205 1427 50  0000 C CNN
+F 2 "" H 3200 1600 50  0000 C CNN
+F 3 "" H 3200 1600 50  0000 C CNN
+	1    3200 1600
+	1    0    0    -1
+$EndComp
+Wire Wire Line
+	1750 2400 1350 2400
+Wire Wire Line
+	1750 2500 1350 2500
+Wire Wire Line
+	2950 2000 3350 2000
+Wire Wire Line
+	2950 1900 3350 1900
+Text Label 1350 2400 0    50   ~ 0
 ~OE_MCU
-Text GLabel 2400 2400 0    50   Input ~ 0
+Text GLabel 1100 2500 0    50   Input ~ 0
 EM_STOP
-Text Label 4500 1800 0    50   ~ 0
+Text Label 3200 1900 0    50   ~ 0
 SCL
-Text Label 4500 1900 0    50   ~ 0
+Text Label 3200 2000 0    50   ~ 0
 SDA
-NoConn ~ 3050 1100
-NoConn ~ 3050 1200
-NoConn ~ 3050 1300
-NoConn ~ 3050 1400
-NoConn ~ 3050 1500
-NoConn ~ 3050 1600
-NoConn ~ 3050 1700
-NoConn ~ 3050 1800
-NoConn ~ 3050 1900
-NoConn ~ 3050 2000
-NoConn ~ 3050 2100
-NoConn ~ 4250 2400
-NoConn ~ 4250 2300
-NoConn ~ 4250 2200
-NoConn ~ 4250 2100
-NoConn ~ 4250 2000
-NoConn ~ 4250 1700
-NoConn ~ 4250 1600
-NoConn ~ 4250 1500
-NoConn ~ 4250 1100
-NoConn ~ 4250 1200
+NoConn ~ 1750 1200
+NoConn ~ 1750 1300
+NoConn ~ 1750 1400
+NoConn ~ 1750 1500
+NoConn ~ 1750 1600
+NoConn ~ 1750 1700
+NoConn ~ 1750 1800
+NoConn ~ 1750 1900
+NoConn ~ 1750 2000
+NoConn ~ 1750 2100
+NoConn ~ 1750 2200
+NoConn ~ 2950 2500
+NoConn ~ 2950 2400
+NoConn ~ 2950 2300
+NoConn ~ 2950 2200
+NoConn ~ 2950 2100
+NoConn ~ 2950 1800
+NoConn ~ 2950 1700
+NoConn ~ 2950 1600
+NoConn ~ 2950 1300
 Wire Wire Line
 	4200 4350 4350 4350
@@
 $EndComp
 Wire Notes Line
-	5400 2950 5400 5100
-Wire Notes Line
 	3450 2950 3450 5100
 Wire Notes Line
@@
 NoConn ~ 9900 2050
 Wire Wire Line
-	3050 2200 2650 2200
-Text Label 2150 2200 0    50   ~ 0
+	1750 2300 1350 2300
+Text Label 850  2300 0    50   ~ 0
 ALERT
 Connection ~ 1800 5250
@@
 L devices:Jumper_NO_Small JP9
 U 1 1 5F60D737
-P 2550 2200
-F 0 "JP9" H 2550 2293 50  0000 C CNN
-F 1 "Jumper_NO_Small" H 2560 2140 50  0001 C CNN
-F 2 "wire_pads:SolderJumper_2mm" H 2550 2150 50  0001 C CNN
-F 3 "" H 2550 2200 50  0000 C CNN
-	1    2550 2200
+P 1250 2300
+F 0 "JP9" H 1250 2393 50  0000 C CNN
+F 1 "Jumper_NO_Small" H 1260 2240 50  0001 C CNN
+F 2 "wire_pads:SolderJumper_2mm" H 1250 2250 50  0001 C CNN
+F 3 "" H 1250 2300 50  0000 C CNN
+	1    1250 2300
 	-1   0    0    1
 $EndComp
@@
 L devices:Jumper_NO_Small JP10
 U 1 1 5F61363A
-P 2550 2400
-F 0 "JP10" H 2550 2493 50  0000 C CNN
-F 1 "Jumper_NO_Small" H 2560 2340 50  0001 C CNN
-F 2 "wire_pads:SolderJumper_2mm" H 2550 2350 50  0001 C CNN
-F 3 "" H 2550 2400 50  0000 C CNN
-	1    2550 2400
+P 1250 2500
+F 0 "JP10" H 1250 2593 50  0000 C CNN
+F 1 "Jumper_NO_Small" H 1260 2440 50  0001 C CNN
+F 2 "wire_pads:SolderJumper_2mm" H 1250 2450 50  0001 C CNN
+F 3 "" H 1250 2500 50  0000 C CNN
+	1    1250 2500
 	-1   0    0    1
 $EndComp
 Wire Wire Line
-	2450 2200 2150 2200
-Wire Wire Line
-	2450 2400 2400 2400
+	1150 2300 850  2300
+Wire Wire Line
+	1150 2500 1100 2500
+Wire Wire Line
+	2950 1200 3100 1200
+Wire Wire Line
+	3100 1200 3100 1050
+$Comp
+L power-supply:+5V #PWR0115
+U 1 1 5F641F07
+P 3100 1050
+F 0 "#PWR0115" H 3100 900 50  0001 C CNN
+F 1 "+5V" H 3115 1223 50  0000 C CNN
+F 2 "" H 3100 1050 50  0000 C CNN
+F 3 "" H 3100 1050 50  0000 C CNN
+	1    3100 1050
+	1    0    0    -1
+$EndComp
+$Comp
+L devices:Label L?
+U 1 1 5F657E7F
+P 6100 900
+F 0 "L?" H 6328 953 60  0000 L CNN
+F 1 "Label" H 6328 847 60  0000 L CNN
+F 2 "" H 6000 1000 60  0000 C CNN
+F 3 "" H 6100 900 60  0000 C CNN
+	1    6100 900
+	1    0    0    -1
+$EndComp
+$Comp
+L devices:Label L?
+U 1 1 5F6586B6
+P 6100 1350
+F 0 "L?" H 6328 1403 60  0000 L CNN
+F 1 "Label" H 6328 1297 60  0000 L CNN
+F 2 "" H 6000 1450 60  0000 C CNN
+F 3 "" H 6100 1350 60  0000 C CNN
+	1    6100 1350
+	1    0    0    -1
+$EndComp
+$Comp
+L devices:Label L?
+U 1 1 5F658BD8
+P 6100 1800
+F 0 "L?" H 6328 1853 60  0000 L CNN
+F 1 "Label" H 6328 1747 60  0000 L CNN
+F 2 "" H 6000 1900 60  0000 C CNN
+F 3 "" H 6100 1800 60  0000 C CNN
+	1    6100 1800
+	1    0    0    -1
+$EndComp
+Wire Notes Line
+	5400 500  5400 5100
 $EndSCHEMATC
