File: kicad/power.sch (KiCad schematic (older format))
At the start: 30 parts, among them P5 WR-TBL_691313710002, U3 LT1117, U4 TPS54335A

Commit message: bom update
Parts:
- C15, C17, C21: value 47 uF -> 47uF
Changed lines of the file:
@@
 P 4400 1800
 F 0 "C15" H 4488 1846 50  0000 L CNN
-F 1 "47 uF" H 4488 1755 50  0000 L CNN
+F 1 "47uF" H 4488 1755 50  0000 L CNN
 F 2 "capacitors:TantalC_SizeD_EIA-7343_Wave" H 4400 1800 50  0001 C CNN
 F 3 "" H 4400 1800 50  0000 C CNN
@@
 P 7400 4600
 F 0 "C21" H 7488 4691 50  0000 L CNN
-F 1 "47 uF" H 7488 4600 50  0000 L CNN
+F 1 "47uF" H 7488 4600 50  0000 L CNN
 F 2 "capacitors:c_elec_8x6.7" H 7488 4509 50  0000 L CNN
 F 3 "" H 7400 4600 50  0000 C CNN
@@
 P 4550 6950
 F 0 "C17" H 4638 7041 50  0000 L CNN
-F 1 "47 uF" H 4638 6950 50  0000 L CNN
+F 1 "47uF" H 4638 6950 50  0000 L CNN
 F 2 "capacitors:c_elec_8x6.7" H 4638 6859 50  0000 L CNN
 F 3 "" H 4550 6950 50  0000 C CNN
